Commit message: history adding to actor

File: simulation/legged_gym/resources/robots/g1_modified/g1_23dof.urdf (robot description, URDF)
Before this commit: robot g1_23dof, 32 links, 31 joints
Links:
- link torso_link: mass 8.562 -> 1.562

Commit message: fix: history actor + ref motion

File: simulation/legged_gym/resources/robots/g1_modified/g1_23dof.urdf (robot description, URDF)
Before this commit: robot g1_23dof, 32 links, 31 joints
Links:
- link torso_link: mass 1.562 -> 9.562

Commit message: history rand

File: simulation/legged_gym/resources/robots/g1_modified/g1_23dof.urdf (robot description, URDF)
Before this commit: robot g1_23dof, 32 links, 31 joints
Links:
- link torso_link: mass 9.562 -> 10.562
